Commit message: duplo brick model stl

File: models/duplo_brick/model.urdf (robot description, URDF)
Before this commit: robot duplo_brick, 1 links, 0 joints
Links:
- link brick: geometry collision box size=0.069 0.032 0.024; visual mesh filename=package://baxter_pick_and_place/models/duplo_brick/meshes/m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
